File: Filtre-de-resolution-MSA-200-Hz/Filtre-de-resolution-MSA-200-Hz.kicad_pcb (KiCad board)
At the start: 2 copper layers, 111 x 55 mm, 35 parts, among them IC1 OPA356, P1 SMA, P2 Connecteur2Pin, P3 SMA, T1 T1-1T-KK81+, T2 T1-1T-KK81+, X1 10.7 MHz, X2 10.7 MHz, X3 10.7 MHz, X4 10.7 MHz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

Commit message: Update project
Update Schematic and PCB
Add a new library
Parts:
- removed Condensateur1, Condensateur2, Condensateur8, Condensateur9: 100 nF, Kicad-Empreintes:condensateur_0805
- removed Condensateur10, Condensateur13, Condensateur3, Condensateur6: 100 pF, Kicad-Empreintes:condensateur_0805
- removed Condensateur11, Condensateur12, Condensateur4, Condensateur5: 220 pF, Kicad-Empreintes:condensateur_0805
- removed Condensateur7: 1µF, Kicad-Empreintes:condensateur_0805
- added C1: 100 nF, Kicad-Empreintes:condensateur_0805, F.Cu at (104.1, 102.2)
- added C10: 100 pF, Kicad-Empreintes:condensateur_0805, F.Cu at (172.7, 84.5)
- added C11: 220 pF, Kicad-Empreintes:condensateur_0805, F.Cu at (172.7, 87.6)
- added C12: 100 pF, Kicad-Empreintes:condensateur_0805, F.Cu at (172.7, 118.1)
- added C13: 220 pF, Kicad-Empreintes:condensateur_0805, F.Cu at (172.7, 121.3)
- added C2: 100 nF, Kicad-Empreintes:condensateur_0805, F.Cu at (185.4, 102.2)
- added C3: 100 pF, Kicad-Empreintes:condensateur_0805, F.Cu at (116.8, 87.6)
- added C4: 220 pF, Kicad-Empreintes:condensateur_0805, F.Cu at (116.8, 84.5)
- added C5: 100 pF, Kicad-Empreintes:condensateur_0805, F.Cu at (116.9, 120.7)
- added C6: 220 pF, Kicad-Empreintes:condensateur_0805, F.Cu at (116.9, 117.5)
- added C7: 1 µF, Kicad-Empreintes:condensateur_0805, F.Cu at (137.2, 83.2)
- added C8: 100 nF, Kicad-Empreintes:condensateur_0805, F.Cu at (135.9, 109.9)
- added C9: 100 nF, Kicad-Empreintes:condensateur_0805, F.Cu at (153.0, 109.9)
- added VG1: ViaGround, Kicad-Empreintes:ViaGround, F.Cu at (159.0, 81.8)
- added VG10: ViaGround, Kicad-Empreintes:ViaGround, F.Cu at (144.8, 118.4)
- added VG11: ViaGround, Kicad-Empreintes:ViaGround, F.Cu at (130.6, 93.5)
- added VG12: ViaGround, Kicad-Empreintes:ViaGround, F.Cu at (130.6, 128.0)
- added VG13: ViaGround, Kicad-Empreintes:ViaGround, F.Cu at (155.4, 97.0)
- added VG14: ViaGround, Kicad-Empreintes:ViaGround, F.Cu at (130.6, 118.4)
- added VG15: ViaGround, Kicad-Empreintes:ViaGround, F.Cu at (149.9, 97.0)
- added VG16: ViaGround, Kicad-Empreintes:ViaGround, F.Cu at (144.8, 111.8)
- added VG17: ViaGround, Kicad-Empreintes:ViaGround, F.Cu at (135.1, 97.0)
- added VG18: ViaGround, Kicad-Empreintes:ViaGround, F.Cu at (159.0, 118.4)
- added VG19: ViaGround, Kicad-Empreintes:ViaGround, F.Cu at (130.6, 100.6)
- added VG2: ViaGround, Kicad-Empreintes:ViaGround, F.Cu at (159.0, 94.0)
- added VG20: ViaGround, Kicad-Empreintes:ViaGround, F.Cu at (144.8, 128.0)
- added VG21: ViaGround, Kicad-Empreintes:ViaGround, F.Cu at (130.6, 123.4)
- added VG22: ViaGround, Kicad-Empreintes:ViaGround, F.Cu at (130.6, 81.8)
- added VG23: ViaGround, Kicad-Empreintes:ViaGround, F.Cu at (130.6, 97.0)
- added VG24: ViaGround, Kicad-Empreintes:ViaGround, F.Cu at (159.0, 128.0)
- added VG25: ViaGround, Kicad-Empreintes:ViaGround, F.Cu at (159.0, 123.4)
- added VG26: ViaGround, Kicad-Empreintes:ViaGround, F.Cu at (139.2, 97.0)
- added VG27: ViaGround, Kicad-Empreintes:ViaGround, F.Cu at (159.0, 104.6)
- added VG28: ViaGround, Kicad-Empreintes:ViaGround, F.Cu at (159.0, 85.9)
- added VG29: ViaGround, Kicad-Empreintes:ViaGround, F.Cu at (144.8, 123.4)
- added VG3: ViaGround, Kicad-Empreintes:ViaGround, F.Cu at (159.0, 89.9)
- added VG30: ViaGround, Kicad-Empreintes:ViaGround, F.Cu at (159.0, 101.1)
- added VG31: ViaGround, Kicad-Empreintes:ViaGround, F.Cu at (130.6, 85.9)
- added VG32: ViaGround, Kicad-Empreintes:ViaGround, F.Cu at (159.0, 77.2)
- added VG4: ViaGround, Kicad-Empreintes:ViaGround, F.Cu at (130.6, 105.2)
- added VG5: ViaGround, Kicad-Empreintes:ViaGround, F.Cu at (130.6, 112.8)
- added VG6: ViaGround, Kicad-Empreintes:ViaGround, F.Cu at (130.6, 89.9)
- added VG7: ViaGround, Kicad-Empreintes:ViaGround, F.Cu at (130.6, 77.2)
- added VG8: ViaGround, Kicad-Empreintes:ViaGround, F.Cu at (144.8, 99.6)
- added VG9: ViaGround, Kicad-Empreintes:ViaGround, F.Cu at (159.0, 112.8)
- moved R2 9.16 mm to (137.2, 88.9), turned to 180 degrees
- moved R1 8.39 mm to (142.9, 88.9), turned to 180 degrees
- moved R6 5.79 mm to (153.0, 106.0)
- moved R3 3.11 mm to (135.9, 102.9)
- moved R4 2.82 mm to (142.9, 83.2)
- moved R7 2.00 mm to (153.0, 102.9)
- moved T2 1.49 mm to (172.7, 102.2)
- moved R5 1.19 mm to (140.3, 109.9)
- moved X7 1.06 mm to (181.0, 92.8)
- moved X8 1.03 mm to (181.0, 113.0)
- moved X2 0.61 mm to (108.0, 112.4)
- moved X5 0.59 mm to (164.5, 92.8)
- moved X6 0.54 mm to (164.5, 113.0)
- moved T1 0.52 mm to (116.8, 102.5)
- moved P2 0.42 mm to (148.0, 77.0)
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Connections:
- net /sheet5D655E65/Input renamed /sheet5D627408/Input
- net /sheet5D655E65/Output renamed /sheet5D627408/Output
Routing:
- net /AmplificateurRF/Input: track 0.00 -> 44.9 mm, vias 0 -> 1
- net GND: track 0.00 -> 34.2 mm, vias 0 -> 10
- net Net-(C9-Pad1): track 0.00 -> 31.5 mm, vias 0 -> 2
- net Net-(C12-Pad1): track 0.00 -> 25.4 mm
- net Net-(C5-Pad1): track 0.00 -> 25.2 mm
- net Net-(C3-Pad2): track 0.00 -> 24.4 mm
- net Net-(C10-Pad2): track 0.00 -> 24.2 mm
- net /sheet5D627408/Input: track 0.00 -> 21.7 mm
- net /sheet5D627408/Output: track 0.00 -> 14.6 mm
- net Net-(C3-Pad1): track 0.00 -> 14.6 mm
- net Net-(C10-Pad1): track 0.00 -> 14.0 mm
- net Net-(C12-Pad2): track 0.00 -> 14.0 mm
- net Net-(IC1-Pad4): track 0.00 -> 13.9 mm
- net Net-(C5-Pad2): track 0.00 -> 13.7 mm
- net /Cellule-Filtre/Input: track 0.00 -> 13.4 mm
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- added copper zone on B.Cu, net GND
- added copper zone on F.Cu, net GND
Other:
- board text added: "+5V"
- board text added: "Alimentation"
- board text added: "Cellule 1"
- board text added: "Cellule 2"
- board text added: "Compensation"
- board text added: "Entrée"
- board text added: "Filtre de résolution 10.7 MHz MSA F1OKU F4HYU"
- board text added: "GND"
- board text added: "Sortie"
