File: Filtre-de-resolution-MSA-200-Hz/Filtre-de-resolution-MSA-200-Hz.sch (KiCad schematic (older format))
At the start: 5 parts, among them P1 SMA, P2 Connecteur2Pin, P3 SMA

Commit message: Update project
Update Schematic and PCB
Add a new library
Parts:
- removed Condensateur1, Condensateur2: 100 nF, Kicad-Empreintes:condensateur_0805, symbol condensateur_0805:C
- added C1, C2: 100 nF, Kicad-Empreintes:condensateur_0805, symbol condensateur_0805:Condensateur
- added VG1, VG10, VG11, VG12, VG13, VG14, VG15, VG16, VG17, VG18, VG19, VG2, VG20, VG21, VG22, VG23, VG24, VG25, VG26, VG27, VG28, VG29, VG3, VG30, VG31, VG32, VG4, VG5, VG6, VG7, VG8, VG9: ViaGround, Kicad-Empreintes:ViaGround, symbol Via-Masse:ViaGround
Connections:
- net Cellule-Filtre/Input: now also C1.2
- net GND: now also VG1.1, VG10.1, VG11.1, VG12.1, VG13.1, VG14.1, VG15.1, VG16.1, VG17.1, VG18.1, VG19.1, VG2.1, VG20.1, VG21.1, VG22.1, VG23.1, VG24.1, VG25.1, VG26.1, VG27.1, VG28.1, VG29.1, VG3.1, VG30.1, VG31.1, VG32.1, VG4.1, VG5.1, VG6.1, VG7.1, VG8.1, VG9.1
- net at P1.1 (In): now also C1.1
- net at P3.1 (In): now also C2.2
- new net sheet5D627408/Output: C2.1
